File: mattduino_uno.sch (EAGLE design)
At the start: 32 parts, among them IC3 CH340G, IC4 LM317MBSTT3, IC5 NX1117C33Z, J4 POWER_JACK, J6 USB_B_PTH, Q2 16MHz, U1 ATMEGA328P_TQFP, Y1 12Mhz

Commit message: missing stuff
Parts:
- removed Q2: 16MHz, SparkFun-Clocks:CRYSTALPTH-HC49UV
- removed R10, R11: 1k, rcl:R-EU_R1206
- added C4: 0.1uF, rcl:C-EUC0603
- added R3: 1M, rcl:R-EU_R0603
- added Y1B: 12Mhz, SparkFun-Clocks:CRYSTAL-8MHZSMD-HC49UP
- added Y2: 16Mhz, SparkFun-Clocks:CRYSTAL-8MHZSMD-HC49UP
- added Y2B: 16MHz, SparkFun-Clocks:CRYSTALPTH-HC49UV
- C1, C10, C12, C13, C14, C2, C8, C9: device rcl:C-EUC1206 -> rcl:C-EUC0603
- R1, R2, R6, R7, R8, R9: device rcl:R-EU_R1206 -> rcl:R-EU_R0603
- RX, TX: device SparkFun-LED:LED1206 -> led:LEDCHIP-LED0603
Connections:
- net N$3 renamed V3
- removed net CH340_RX: IC3.RX, R11.1
- removed net CH340_TX: IC3.TX, R10.1
- net +5V: now also C4.1
- net 328_OSC1: now also Y2.1, Y2B.1; no longer Q2.1
- net 328_OSC2: now also Y2.2, Y2B.2; no longer Q2.2
- net GND: now also C4.2
- net IO11/MOSI: now also B2.MOSI; no longer B2.MISO
- net IO12/MISO: now also B2.MISO; no longer B2.MOSI
- net OSCI: now also R3.1, Y1B.1
- net OSCO: now also R3.2, Y1B.2
- net RX: now also IC3.TX; no longer R10.2
- net TX: now also IC3.RX; no longer R11.2
Other:
- moved on the sheet: C1, C12, C13, C2, Y1
