File: mattduino_uno.v7.brd (EAGLE design)
At the start: 68.6 x 53.3 mm, 32 parts, among them IC3 CH340G, IC4 LM317MBSTT3, IC5 NX1117C33Z, J4 POWER_JACK, J6 USB_B_PTH, Q2 16MHz, U1 ATMEGA328P_TQFP, Y1 12Mhz

Commit message: missing stuff
Parts:
- removed Q2: 16MHz, SparkFun-Clocks:HC49U
- added Y1B: 12Mhz, SparkFun-Clocks@1:HC49UP
- added Y2: 16Mhz, SparkFun-Clocks@1:HC49UP
- added Y2B: 16MHz, SparkFun-Clocks:HC49U
- moved R1 8.29 mm to (52.8, 41.1), turned to 180 degrees
- moved C1 7.77 mm to (55.6, 38.6), turned to 180 degrees
- moved C2 4.54 mm to (50.0, 38.6), turned to 0 degrees
Connections:
- net 328_OSC1: now also Y2.1, Y2B.1; no longer Q2.1
- net 328_OSC2: now also Y2.2, Y2B.2; no longer Q2.2
- net IO11/MOSI: now also B2.MOSI; no longer B2.MISO
- net IO12/MISO: now also B2.MISO; no longer B2.MOSI
- net OSCI: now also Y1B.1
- net OSCO: now also Y1B.2
Routing:
- net IO11/MOSI: track 49.5 -> 55.8 mm
- net IO3: track 34.3 -> 38.5 mm
- net IO4: track 34.6 -> 38.3 mm
- net IO2: track 39.1 -> 42.2 mm
- net USB-: track 17.9 -> 20.6 mm
- net IO12/MISO: track 54.9 -> 52.2 mm
- net OSCO: track 8.96 -> 11.4 mm
- net OSCI: track 13.2 -> 15.6 mm
- net USB+: track 20.7 -> 23.0 mm
- net RX: track 111.6 -> 109.4 mm
- net 328_OSC1: track 23.7 -> 22.5 mm
- net 328_OSC2: track 16.5 -> 17.3 mm
- net TX: track 100.9 -> 101.4 mm
- net +5V: track 190.1 -> 190.6 mm
