File: mattduino_uno.v7.sch (EAGLE design)
At the start: 32 parts, among them IC3 CH340G, IC4 LM317MBSTT3, IC5 NX1117C33Z, J4 POWER_JACK, J6 USB_B_PTH, Q2 16MHz, U1 ATMEGA328P_TQFP, Y1 12Mhz

Commit message: missing stuff
Parts:
- removed Q2: 16MHz, SparkFun-Clocks:CRYSTALPTH-HC49UV
- added Y1B: 12Mhz, SparkFun-Clocks@1:CRYSTAL-8MHZSMD-HC49UP
- added Y2: 16Mhz, SparkFun-Clocks@1:CRYSTAL-8MHZSMD-HC49UP
- added Y2B: 16MHz, SparkFun-Clocks:CRYSTALPTH-HC49UV
Connections:
- net 328_OSC1: now also Y2.1, Y2B.1; no longer Q2.1
- net 328_OSC2: now also Y2.2, Y2B.2; no longer Q2.2
- net IO11/MOSI: now also B2.MOSI; no longer B2.MISO
- net IO12/MISO: now also B2.MISO; no longer B2.MOSI
- net OSCI: now also Y1B.1
- net OSCO: now also Y1B.2
Other:
- moved on the sheet: C1, C2
